Commit message: first runnalbe version, still use mapping/odometry_incremental

File: config/robot.urdf.xacro (robot description, xacro)
@@ -2,5 +2,11 @@
 <robot name="lio" xmlns:xacro="http://tixiaoshan.github.io/">
   <xacro:property name="PI" value="3.1415926535897931" />
+  <link name="map"></link>
   <link name="odom"></link>
+  <joint name="map_joint" type="fixed">
+    <origin xyz="0.0 0.0 0.0" rpy="0.0 0.0 0.0"/>
+    <parent link="map"/>
+    <child link="odom"/>
+  </joint>
   <link name="base_link"></link>
   <joint name="odom_joint" type="continuous">
@@ -9,32 +15,8 @@
     <child link="base_link"/>
   </joint>
-  <link name="lidar_link"></link>
-  <joint name="lidar_joint" type="fixed">
-    <parent link="base_link" />
-    <child link="lidar_link" />
-    <origin xyz="0 0 0" rpy="0 0 0" />
-  </joint>
-  <link name="velodyne"></link>
-  <joint name="velodyne_joint" type="fixed">
-    <parent link="base_link" />
-    <child link="velodyne" />
-    <origin xyz="0 0 0" rpy="0 0 0" />
-  </joint>
-  <link name="laser_data_frame"></link>
-  <joint name="laser_data_frame_joint" type="fixed">
-    <parent link="base_link" />
-    <child link="laser_data_frame" />
-    <origin xyz="0 0 0" rpy="0 0 0" />
-  </joint>
   <link name="imu_link"> </link>
   <joint name="imu_joint" type="fixed">
     <parent link="base_link" />
     <child link="imu_link" />
-    <origin xyz="0 0 0" rpy="0 0 0" />
-  </joint>
-  <link name="laser_sensor_frame"> </link>
-  <joint name="laser_joint" type="fixed">
-    <parent link="imu_link" />
-    <child link="laser_sensor_frame" />
     <origin xyz="0 0 0" rpy="0 0 0" />
   </joint>
